Commit message: Added D48-specific urdf and xacro files

File: flir_ptu_description/urdf/d48.urdf.xacro (robot description, xacro)
@@ -1,4 +1,4 @@
 <?xml version="1.0"?>
-<robot name="ptu_d46"
+<robot name="ptu_d48"
        xmlns:xacro="http://ros.org/wiki/xacro">
   <xacro:property name="pan_velocity" value="1.0" />
@@ -8,8 +8,7 @@
   <xacro:property name="tilt_down_range" value="0.82" />
   <xacro:property name="joint_effort" value="30" />
-  <xacro:macro name="d46_stepper_module"
-               params="ptu_name joint_name">
-    <link name="${ptu_name}_${joint_name}_link">
-      <!-- <inertial>
+  <xacro:macro name="ptu_d48" params="name">
+    <link name="${name}_base_link">
+			<!-- <inertial>
         <mass value="0.65" />
         <inertia ... ? />
@@ -20,26 +19,39 @@
         </material>
         <geometry>
-          <box size="0.045 0.065 0.044" />
+					<mesh filename="package://flir_ptu_description/urdf/meshes/d48_ptu_base.STL"/>
         </geometry>
-        <origin xyz="0 0.011 0" />
+        <origin xyz="0 0 0" />
       </visual>
+		</link>
+    <link name="${name}_pan_link">
+			<!-- <inertial>
+        <mass value="0.65" />
+        <inertia ... ? />
+      </inertial> -->
       <visual>
+        <material name="ptu_body_color">
+          <color rgba="0.3 0.3 0.3 1.0" />
+        </material>
         <geometry>
-          <box size="0.046 0.044 0.044" />
+					<mesh filename="package://flir_ptu_description/urdf/meshes/d48_ptu_body.STL"/>
         </geometry>
-        <origin xyz="-0.045 0.0215 0" />
+        <origin xyz="0 0 0" />
       </visual>
+		</link>
+    <link name="${name}_tilt_link">
+			<!-- <inertial>
+        <mass value="0.65" />
+        <inertia ... ? />
+      </inertial> -->
       <visual>
+        <material name="ptu_body_color">
+          <color rgba="0.3 0.3 0.3 1.0" />
+        </material>
         <geometry>
-          <cylinder length="0.015" radius="0.005" />
+					<mesh filename="package://flir_ptu_description/urdf/meshes/d48_ptu_mount.STL"/>
         </geometry>
-        <origin xyz="-0.074 0.021 0" rpy="0 1.57 0" />
+        <origin xyz="0 0 0" />
       </visual>
-    </link>
-  </xacro:macro>
-  <xacro:macro name="ptu_d46" params="name">
-    <d46_stepper_module ptu_name="${name}" joint_name="pan" />
-    <d46_stepper_module ptu_name="${name}" joint_name="tilt" />
-    <link name="${name}_base_link" />
+		</link>
     <link name="${name}_tilted_link" />
     <link name="${name}_mount_link" />
@@ -49,12 +61,12 @@
       <parent link="${name}_base_link"/>
       <child link="${name}_pan_link"/>
-      <origin xyz="0 -0.011 0.022"/>
+      <origin xyz="0 0 0.092"/>
     </joint>
     <!-- The pan joint -->
     <joint name="${name}_pan" type="revolute">
       <parent link="${name}_pan_link" />
-      <origin xyz="0 0 0.066" rpy="-1.5708 0 0" />
+      <origin xyz="0 0 0.13" />
       <child link="${name}_tilt_link" />
-      <axis xyz="0 1 0" rpy="0 0 0" />
+      <axis xyz="0 1 0" />
       <limit lower="${pan_range}" upper="${-pan_range}"
              effort="${joint_effort}" velocity="${pan_velocity}" />
@@ -63,5 +75,5 @@
     <joint name="${name}_tilt" type="revolute">
       <parent link="${name}_tilt_link" />
-      <origin xyz="0 0 0" rpy="-1.5708 0 0" />
+      <origin xyz="0 0 0" />
       <child link="${name}_tilted_link" />
       <axis xyz="0 1 0" />
@@ -73,5 +85,5 @@
       <parent link="${name}_tilted_link"/>
       <child link="${name}_mount_link"/>
-      <origin xyz="0 0 -0.03912" rpy="3.1416 0 0" />
+      <origin xyz="0 0 0.046" />
     </joint>
   </xacro:macro>

Commit message: More reliability fixes, corrected d48 urdf

File: flir_ptu_description/urdf/d48.urdf.xacro (robot description, xacro)
@@ -10,5 +10,5 @@
   <xacro:macro name="ptu_d48" params="name">
     <link name="${name}_base_link">
-			<!-- <inertial>
+      <!-- <inertial>
         <mass value="0.65" />
         <inertia ... ? />
@@ -19,11 +19,11 @@
         </material>
         <geometry>
-					<mesh filename="package://flir_ptu_description/urdf/meshes/d48_ptu_base.STL"/>
+          <mesh filename="package://flir_ptu_description/urdf/meshes/d48_ptu_base.STL"/>
         </geometry>
         <origin xyz="0 0 0" />
       </visual>
-		</link>
+    </link>
     <link name="${name}_pan_link">
-			<!-- <inertial>
+      <!-- <inertial>
         <mass value="0.65" />
         <inertia ... ? />
@@ -34,11 +34,11 @@
         </material>
         <geometry>
-					<mesh filename="package://flir_ptu_description/urdf/meshes/d48_ptu_body.STL"/>
+          <mesh filename="package://flir_ptu_description/urdf/meshes/d48_ptu_body.STL"/>
         </geometry>
         <origin xyz="0 0 0" />
       </visual>
-		</link>
+    </link>
     <link name="${name}_tilt_link">
-			<!-- <inertial>
+      <!-- <inertial>
         <mass value="0.65" />
         <inertia ... ? />
@@ -49,33 +49,26 @@
         </material>
         <geometry>
-					<mesh filename="package://flir_ptu_description/urdf/meshes/d48_ptu_mount.STL"/>
+          <mesh filename="package://flir_ptu_description/urdf/meshes/d48_ptu_mount.STL"/>
         </geometry>
         <origin xyz="0 0 0" />
       </visual>
-		</link>
-    <link name="${name}_tilted_link" />
+    </link>
     <link name="${name}_mount_link" />
     <!-- There's an offset between the origin of the pan joint and the origin of
          the overall device, which is between the mounting screws on its base. -->
-    <joint name="${name}_base" type="fixed">
+    <joint name="${name}_pan" type="revolute">
       <parent link="${name}_base_link"/>
       <child link="${name}_pan_link"/>
       <origin xyz="0 0 0.092"/>
+      <axis xyz="0 0 -1" />
+      <limit lower="${pan_range}" upper="${-pan_range}"
+             effort="${joint_effort}" velocity="${pan_velocity}" />
     </joint>
     <!-- The pan joint -->
-    <joint name="${name}_pan" type="revolute">
+    <joint name="${name}_tilt" type="revolute">
       <parent link="${name}_pan_link" />
       <origin xyz="0 0 0.13" />
       <child link="${name}_tilt_link" />
-      <axis xyz="0 1 0" />
-      <limit lower="${pan_range}" upper="${-pan_range}"
-             effort="${joint_effort}" velocity="${pan_velocity}" />
-    </joint>
-    <!-- The tilt joint -->
-    <joint name="${name}_tilt" type="revolute">
-      <parent link="${name}_tilt_link" />
-      <origin xyz="0 0 0" />
-      <child link="${name}_tilted_link" />
-      <axis xyz="0 1 0" />
+      <axis xyz="0 -1 0" />
       <limit lower="${-tilt_down_range}" upper="${tilt_up_range}"
              effort="${joint_effort}" velocity="${tilt_velocity}" />
@@ -83,5 +76,5 @@
     <!-- Fixed joint to provide a convenient attachment point for accessories. -->
     <joint name="${name}_mount" type="fixed">
-      <parent link="${name}_tilted_link"/>
+      <parent link="${name}_tilt_link"/>
       <child link="${name}_mount_link"/>
       <origin xyz="0 0 0.046" />
