Commit message: General fixes, especially install macros, and building the example urdf at make time.

File: flir_ptu_description/urdf/d46.urdf.xacro (robot description, xacro)
@@ -44,7 +44,7 @@
     <link name="${name}_tilted_link" />
     <link name="${name}_mount_link" />
-    <!-- There's a offset between the origin of the pan joint and the origin of
-         the overall device. -->
-    <joint name="${name}_base_to_pan" type="fixed">
+    <!-- There's an offset between the origin of the pan joint and the origin of
+         the overall device, which is between the mounting screws on its base. -->
+    <joint name="${name}_base" type="fixed">
       <parent link="${name}_base_link"/>
       <child link="${name}_pan_link"/>
@@ -52,5 +52,5 @@
     </joint>
     <!-- The pan joint -->
-    <joint name="${name}_pan_to_tilt" type="revolute">
+    <joint name="${name}_pan" type="revolute">
       <parent link="${name}_pan_link" />
       <origin xyz="0 0 0.066" rpy="-1.5708 0 0" />
@@ -61,5 +61,5 @@
     </joint>
     <!-- The tilt joint -->
-    <joint name="${name}_tilt_to_tilted" type="revolute">
+    <joint name="${name}_tilt" type="revolute">
       <parent link="${name}_tilt_link" />
       <origin xyz="0 0 0" rpy="-1.5708 0 0" />
@@ -70,5 +70,5 @@
     </joint>
     <!-- Fixed joint to provide a convenient attachment point for accessories. -->
-    <joint name="${name}_tilted_to_mount" type="fixed">
+    <joint name="${name}_mount" type="fixed">
       <parent link="${name}_tilted_link"/>
       <child link="${name}_mount_link"/>

Commit message: Reverse pan joint direction.
Per #15.

File: flir_ptu_description/urdf/d46.urdf.xacro (robot description, xacro)
@@ -56,5 +56,5 @@
       <origin xyz="0 0 0.066" rpy="-1.5708 0 0" />
       <child link="${name}_tilt_link" />
-      <axis xyz="0 1 0" rpy="0 0 0" />
+      <axis xyz="0 -1 0" rpy="3.14159 0 0" />
       <limit lower="${pan_range}" upper="${-pan_range}"
              effort="${joint_effort}" velocity="${pan_velocity}" />

Commit message: Added transmissions and inertial elements for sim

File: flir_ptu_description/urdf/d46.urdf.xacro (robot description, xacro)
@@ -11,8 +11,9 @@
                params="ptu_name joint_name">
     <link name="${ptu_name}_${joint_name}_link">
-      <!-- <inertial>
+      <inertial>
         <mass value="0.65" />
-        <inertia ... ? />
-      </inertial> -->
+        <origin xyz="0 0 0" rpy="0 0 0" />
+        <inertia ixx="0.0001" ixy="0" ixz="0" iyy="0.0001" iyz="0" izz="0.0001" />
+      </inertial>
       <visual>
         <material name="ptu_body_color">
@@ -37,4 +38,18 @@
       </visual>
     </link>
+    <gazebo reference="${ptu_name}_${joint_name}_link">
+        <material>Gazebo/DarkGrey</material>
+    </gazebo>
+  </xacro:macro>
+  <xacro:macro name="d46_transmission" params="name">
+    <transmission name="${name}_trans">
+      <type>transmission_interface/SimpleTransmission</type>
+      <joint name="${name}">
+        <hardwareInterface>PositionJointInterface</hardwareInterface>
+      </joint>
+      <actuator name="${name}_motor">
+        <mechanicalReduction>1</mechanicalReduction>
+      </actuator>
+    </transmission>
   </xacro:macro>
   <xacro:macro name="ptu_d46" params="name">
@@ -60,4 +75,5 @@
              effort="${joint_effort}" velocity="${pan_velocity}" />
     </joint>
+    <d46_transmission name="${name}_pan" />
     <!-- The tilt joint -->
     <joint name="${name}_tilt" type="revolute">
@@ -69,4 +85,5 @@
              effort="${joint_effort}" velocity="${tilt_velocity}" />
     </joint>
+    <d46_transmission name="${name}_tilt" />
     <!-- Fixed joint to provide a convenient attachment point for accessories. -->
     <joint name="${name}_mount" type="fixed">

Commit message: added mesh to visual so openrave can view it, added in transmissions

File: flir_ptu_description/urdf/d46.urdf.xacro (robot description, xacro)
@@ -20,21 +20,27 @@
           <color rgba="0.3 0.3 0.3 1.0" />
         </material>
+        <origin xyz="-0.0295 0.011 0" rpy="3.14 0 0" />
+        <geometry>
+          <mesh filename="package://flir_ptu_description/meshes/flir-ptu-simple.stl"/>
+        </geometry>
+      </visual>
+      <collision>
         <geometry>
           <box size="0.045 0.065 0.044" />
         </geometry>
         <origin xyz="0 0.011 0" />
-      </visual>
-      <visual>
+      </collision>
+      <collision>
         <geometry>
           <box size="0.046 0.044 0.044" />
         </geometry>
         <origin xyz="-0.045 0.0215 0" />
-      </visual>
-      <visual>
+      </collision>
+      <collision>
         <geometry>
           <cylinder length="0.015" radius="0.005" />
         </geometry>
         <origin xyz="-0.074 0.021 0" rpy="0 1.57 0" />
-      </visual>
+      </collision>
     </link>
     <gazebo reference="${ptu_name}_${joint_name}_link">
@@ -72,5 +78,5 @@
       <child link="${name}_tilt_link" />
       <axis xyz="0 -1 0" rpy="3.14159 0 0" />
-      <limit lower="${pan_range}" upper="${-pan_range}"
+      <limit lower="${-pan_range}" upper="${pan_range}"
              effort="${joint_effort}" velocity="${pan_velocity}" />
     </joint>

Commit message: Fix gazebo errors

File: flir_ptu_description/urdf/d46.urdf.xacro (robot description, xacro)
@@ -62,7 +62,17 @@
     <d46_stepper_module ptu_name="${name}" joint_name="pan" />
     <d46_stepper_module ptu_name="${name}" joint_name="tilt" />
-    <link name="${name}_base_link" />
-    <link name="${name}_tilted_link" />
-    <link name="${name}_mount_link" />
+    <link name="${name}_base_link">
+<inertial>
+			<mass value="2e-06"/>
+			<inertia ixx="1.1e-09" ixy="0" ixz="0" iyy="1.1e-09" iyz="0" izz="1.1e-09"/>
+		</inertial>
+    </link>
+    <link name="${name}_tilted_link"/>
+    <link name="${name}_mount_link">
+<inertial>
+			<mass value="2e-06"/>
+			<inertia ixx="1.1e-09" ixy="0" ixz="0" iyy="1.1e-09" iyz="0" izz="1.1e-09"/>
+		</inertial>
+    </link>
     <!-- There's an offset between the origin of the pan joint and the origin of
          the overall device, which is between the mounting screws on its base. -->

Commit message: Revert "Fix gazebo errors"

File: flir_ptu_description/urdf/d46.urdf.xacro (robot description, xacro)
@@ -62,17 +62,7 @@
     <d46_stepper_module ptu_name="${name}" joint_name="pan" />
     <d46_stepper_module ptu_name="${name}" joint_name="tilt" />
-    <link name="${name}_base_link">
-<inertial>
-			<mass value="2e-06"/>
-			<inertia ixx="1.1e-09" ixy="0" ixz="0" iyy="1.1e-09" iyz="0" izz="1.1e-09"/>
-		</inertial>
-    </link>
-    <link name="${name}_tilted_link"/>
-    <link name="${name}_mount_link">
-<inertial>
-			<mass value="2e-06"/>
-			<inertia ixx="1.1e-09" ixy="0" ixz="0" iyy="1.1e-09" iyz="0" izz="1.1e-09"/>
-		</inertial>
-    </link>
+    <link name="${name}_base_link" />
+    <link name="${name}_tilted_link" />
+    <link name="${name}_mount_link" />
     <!-- There's an offset between the origin of the pan joint and the origin of
          the overall device, which is between the mounting screws on its base. -->

Commit message: Fixed spaces, fixed gazebo errors about inertia

File: flir_ptu_description/urdf/d46.urdf.xacro (robot description, xacro)
@@ -62,7 +62,17 @@
     <d46_stepper_module ptu_name="${name}" joint_name="pan" />
     <d46_stepper_module ptu_name="${name}" joint_name="tilt" />
-    <link name="${name}_base_link" />
-    <link name="${name}_tilted_link" />
-    <link name="${name}_mount_link" />
+    <link name="${name}_base_link">
+       <inertial>
+            <mass value="2e-06"/>
+            <inertia ixx="1.1e-09" ixy="0" ixz="0" iyy="1.1e-09" iyz="0" izz="1.1e-09"/>
+        </inertial>
+    </link>
+    <link name="${name}_tilted_link"/>
+    <link name="${name}_mount_link">
+        <inertial>
+            <mass value="2e-06"/>
+            <inertia ixx="1.1e-09" ixy="0" ixz="0" iyy="1.1e-09" iyz="0" izz="1.1e-09"/>
+        </inertial>
+    </link>
     <!-- There's an offset between the origin of the pan joint and the origin of
          the overall device, which is between the mounting screws on its base. -->

Commit message: Add pan offset for centering joint based on calibration

File: flir_ptu_description/urdf/d46.urdf.xacro (robot description, xacro)
@@ -58,5 +58,5 @@
     </transmission>
   </xacro:macro>
-  <xacro:macro name="ptu_d46" params="name">
+  <xacro:macro name="ptu_d46" params="name pan_offset:=0.0">
     <d46_stepper_module ptu_name="${name}" joint_name="pan" />
     <d46_stepper_module ptu_name="${name}" joint_name="tilt" />
@@ -84,5 +84,5 @@
     <joint name="${name}_pan" type="revolute">
       <parent link="${name}_pan_link" />
-      <origin xyz="0 0 0.066" rpy="-1.5708 0 0" />
+      <origin xyz="0 0 0.066" rpy="-1.5708 0 ${pan_offset}" />
       <child link="${name}_tilt_link" />
       <axis xyz="0 -1 0" rpy="3.14159 0 0" />

Commit message: Updated PTU mesh geometry

File: flir_ptu_description/urdf/d46.urdf.xacro (robot description, xacro)
@@ -7,44 +7,4 @@
   <xacro:property name="tilt_down_range" value="0.82" />
   <xacro:property name="joint_effort" value="30" />
-  <xacro:macro name="d46_stepper_module"
-               params="ptu_name joint_name">
-    <link name="${ptu_name}_${joint_name}_link">
-      <inertial>
-        <mass value="0.65" />
-        <origin xyz="0 0 0" rpy="0 0 0" />
-        <inertia ixx="0.0001" ixy="0" ixz="0" iyy="0.0001" iyz="0" izz="0.0001" />
-      </inertial>
-      <visual>
-        <material name="ptu_body_color">
-          <color rgba="0.3 0.3 0.3 1.0" />
-        </material>
-        <origin xyz="-0.0295 0.011 0" rpy="3.14 0 0" />
-        <geometry>
-          <mesh filename="package://flir_ptu_description/meshes/flir-ptu-simple.stl"/>
-        </geometry>
-      </visual>
-      <collision>
-        <geometry>
-          <box size="0.045 0.065 0.044" />
-        </geometry>
-        <origin xyz="0 0.011 0" />
-      </collision>
-      <collision>
-        <geometry>
-          <box size="0.046 0.044 0.044" />
-        </geometry>
-        <origin xyz="-0.045 0.0215 0" />
-      </collision>
-      <collision>
-        <geometry>
-          <cylinder length="0.015" radius="0.005" />
-        </geometry>
-        <origin xyz="-0.074 0.021 0" rpy="0 1.57 0" />
-      </collision>
-    </link>
-    <gazebo reference="${ptu_name}_${joint_name}_link">
-        <material>Gazebo/DarkGrey</material>
-    </gazebo>
-  </xacro:macro>
   <xacro:macro name="d46_transmission" params="name">
     <transmission name="${name}_trans">
@@ -59,6 +19,50 @@
   </xacro:macro>
   <xacro:macro name="ptu_d46" params="name pan_offset:=0.0">
-    <d46_stepper_module ptu_name="${name}" joint_name="pan" />
-    <d46_stepper_module ptu_name="${name}" joint_name="tilt" />
+    <link name="${name}_tilt_link">
+      <inertial>
+        <mass value="0.65" />
+        <origin xyz="0 0 0" rpy="0 0 0" />
+        <inertia ixx="0.0001" ixy="0" ixz="0" iyy="0.0001" iyz="0" izz="0.0001" />
+      </inertial>
+      <visual>
+        <material name="ptu_body_color">
+          <color rgba="0.3 0.3 0.3 1.0" />
+        </material>
+        <geometry>
+          <mesh filename="package://flir_ptu_description/meshes/flir-ptu-tilt-motor.stl"/>
+        </geometry>
+      </visual>
+      <collision>
+        <geometry>
+          <mesh filename="package://flir_ptu_description/meshes/flir-ptu-tilt-motor-collision.stl"/>
+        </geometry>
+      </collision>
+    </link>
+    <gazebo reference="${name}_tilt_link">
+        <material>Gazebo/DarkGrey</material>
+    </gazebo>
+    <link name="${name}_pan_link">
+      <inertial>
+        <mass value="0.65" />
+        <origin xyz="0 0 0" rpy="0 0 0" />
+        <inertia ixx="0.0001" ixy="0" ixz="0" iyy="0.0001" iyz="0" izz="0.0001" />
+      </inertial>
+      <visual>
+        <material name="ptu_body_color">
+          <color rgba="0.3 0.3 0.3 1.0" />
+        </material>
+        <geometry>
+          <mesh filename="package://flir_ptu_description/meshes/flir-ptu-pan-motor.stl"/>
+        </geometry>
+      </visual>
+      <collision>
+        <geometry>
+          <mesh filename="package://flir_ptu_description/meshes/flir-ptu-pan-motor-collision.stl"/>
+        </geometry>
+      </collision>
+    </link>
+    <gazebo reference="${name}_pan_link">
+        <material>Gazebo/DarkGrey</material>
+    </gazebo>
     <link name="${name}_base_link">
        <inertial>
@@ -67,5 +71,19 @@
         </inertial>
     </link>
-    <link name="${name}_tilted_link"/>
+    <link name="${name}_tilted_link">
+      <visual>
+        <material name="ptu_body_color">
+          <color rgba="0.3 0.3 0.3 1.0" />
+        </material>
+        <geometry>
+          <mesh filename="package://flir_ptu_description/meshes/flir-ptu-camera-mount.stl"/>
+        </geometry>
+      </visual>
+      <collision>
+        <geometry>
+          <mesh filename="package://flir_ptu_description/meshes/flir-ptu-camera-mount.stl"/>
+        </geometry>
+      </collision>
+    </link>
     <link name="${name}_mount_link">
         <inertial>
@@ -74,15 +92,13 @@
         </inertial>
     </link>
-    <!-- There's an offset between the origin of the pan joint and the origin of
-         the overall device, which is between the mounting screws on its base. -->
     <joint name="${name}_base" type="fixed">
       <parent link="${name}_base_link"/>
       <child link="${name}_pan_link"/>
-      <origin xyz="0 -0.011 0.022"/>
+      <origin xyz="0 0 0"/>
     </joint>
     <!-- The pan joint -->
     <joint name="${name}_pan" type="revolute">
       <parent link="${name}_pan_link" />
-      <origin xyz="0 0 0.066" rpy="-1.5708 0 ${pan_offset}" />
+      <origin xyz="0 -0.00955 0.046774" rpy="-1.5708 0 ${pan_offset}" />
       <child link="${name}_tilt_link" />
       <axis xyz="0 -1 0" rpy="3.14159 0 0" />
@@ -94,5 +110,5 @@
     <joint name="${name}_tilt" type="revolute">
       <parent link="${name}_tilt_link" />
-      <origin xyz="0 0 0" rpy="-1.5708 0 0" />
+      <origin xyz="0 -0.043713 0" rpy="-1.5708 0 0" />
       <child link="${name}_tilted_link" />
       <axis xyz="0 1 0" />
@@ -105,5 +121,5 @@
       <parent link="${name}_tilted_link"/>
       <child link="${name}_mount_link"/>
-      <origin xyz="0 0 -0.03912" rpy="3.1416 0 0" />
+      <origin xyz="0 0 -0.039116" rpy="3.1416 0 0" />
     </joint>
   </xacro:macro>

Commit message: Fix tilted_link inertia (#42)

File: flir_ptu_description/urdf/d46.urdf.xacro (robot description, xacro)
@@ -72,4 +72,9 @@
     </link>
     <link name="${name}_tilted_link">
+      <inertial>
+        <mass value="2e-06"/>
+        <origin xyz="0 0 0" rpy="0 0 0" />
+        <inertia ixx="1.1e-09" ixy="0" ixz="0" iyy="1.1e-09" iyz="0" izz="1.1e-09"/>
+      </inertial>
       <visual>
         <material name="ptu_body_color">
